File: discipline-pcb.kicad_pcb (KiCad board)
At the start: 2 copper layers, 304.9 x 122.8 mm, 197 parts, among them J1 AVR-ISP-6, SW1 KEYSW, SW10 KEYSW, SW11 KEYSW, SW12 KEYSW, SW13 KEYSW, SW14 KEYSW, SW15 KEYSW, SW16 KEYSW, SW17 KEYSW, SW18 KEYSW, SW19 KEYSW, SW2 KEYSW, SW20 KEYSW, SW21 KEYSW, SW22 KEYSW, SW23 KEYSW, SW24 KEYSW, SW25 KEYSW, SW26 KEYSW, SW27 KEYSW, SW28 KEYSW, SW29 KEYSW, SW3 KEYSW, SW30 KEYSW, SW31 KEYSW, SW32 KEYSW, SW33 KEYSW, SW34 KEYSW, SW35 KEYSW, SW36 KEYSW, SW37 KEYSW, SW38 KEYSW, SW39 KEYSW, SW4 KEYSW, SW40 KEYSW, SW41 KEYSW, SW42 KEYSW, SW43 KEYSW, SW44 KEYSW, SW45 KEYSW, SW46 KEYSW, SW47 KEYSW, SW48 KEYSW, SW49 KEYSW, SW5 KEYSW, SW50 KEYSW, SW51 KEYSW, SW52 KEYSW, SW53 KEYSW, SW54 KEYSW, SW55 KEYSW, SW56 KEYSW, SW57 KEYSW, SW58 KEYSW, SW59 KEYSW, SW6 KEYSW, SW60 KEYSW, SW61 KEYSW, SW62 KEYSW, SW63 KEYSW, SW64 KEYSW, SW65 KEYSW, SW66 KEYSW, SW67 KEYSW, SW68 KEYSW, SW69 KEYSW, SW7 KEYSW, SW70 KEYSW, SW71 KEYSW, SW72 KEYSW, SW73 KEYSW, SW74 KEYSW, SW75 KEYSW, SW76 KEYSW, SW77 KEYSW, SW78 KEYSW, SW8 KEYSW, SW9 KEYSW, U1 ATmega32A-PU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

Commit message: Discipline hs
Parts:
- removed D71: , cftkb:D_DO-35_SOD27_P5.08mm_Horizontal
- removed ST72: 7U, cftkb:MX-7U-Stabilizer
- removed SW69, SW78: KEYSW, cftkb:SW_Cherry_MX1A_1.25u_PCBNOSCREEN
- removed SW70, SW71, SW73, SW74: KEYSW, cftkb:SW_Cherry_MX1A_1.50u_PCBNOSCREEN
- removed SW72, SW75, SW77: KEYSW, cftkb:SW_Cherry_MX1A_1.00u_PCB-NOSCREEN
- removed SW76: KEYSW, cftkb:SW_Cherry_MX1A_ISOEnter_PCB_ReversedStabilizer
- SW1, SW10, SW11, SW12, SW13, SW15, SW17, SW18, SW19, SW2, SW20, SW21, SW22, SW23, SW24, SW25, SW26, SW27, SW28, SW3, SW30, SW32, SW33, SW34, SW35, SW36, SW37, SW38, SW39, SW4, SW40, SW41, SW42, SW44, SW46, SW47, SW48, SW49, SW5, SW50, SW51, SW52, SW53, SW54, SW55, SW57, SW58, SW6, SW62, SW65, SW66, SW67, SW68, SW7, SW8, SW9: footprint cftkb:SW_Cherry_MX1A_1.00u_PCB-NOSCREEN -> bankkis_lib:MX_ALPS_HotSwap_1U
- SW14: footprint cftkb:SW_Cherry_MX1A_2.00u_PCBNOSCREEN -> bankkis_lib:MX_ALPS_HotSwap_2U
- SW16, SW29: footprint cftkb:SW_Cherry_MX1A_1.50u_PCBNOSCREEN -> bankkis_lib:MX_ALPS_HotSwap_1.5U
- SW31, SW56: footprint cftkb:SW_Cherry_MX1A_1.75u_PCBNOSCREEN -> bankkis_lib:MX_ALPS_HotSwap_1.75U
- SW45: footprint cftkb:SW_Cherry_MX1A_2.25u_PCBNOSCREEN -> bankkis_lib:MX_ALPS_HotSwap_2.25U
- SW59, SW60, SW61: footprint cftkb:SW_Cherry_MX1A_1.25u_PCBNOSCREEN -> bankkis_lib:MX_ALPS_HotSwap_1.25U
- SW63, SW64: footprint cftkb:SW_Cherry_MX1A_1.25u_PCBNOSCREEN -> bankkis_lib:MX_ALPS_HotSwap_1U
Routing:
- net row3: track 404.8 -> 290.5 mm, vias 7 -> 3
- net GND: track 223.5 -> 173.8 mm, vias 48 -> 49
- net col14: track 107.8 -> 138.4 mm
- net Net-(D29-Pad2): track 127.9 -> 157.1 mm
- net Net-(D57-Pad2): track 152.2 -> 180.1 mm
- net Net-(D43-Pad2): track 153.6 -> 179.0 mm
- net Net-(D35-Pad2): track 75.5 -> 100.7 mm
- net Net-(D56-Pad2): track 146.5 -> 170.6 mm
- net Net-(D36-Pad2): track 83.2 -> 107.2 mm
- net Net-(D64-Pad2): track 188.7 -> 212.5 mm
- net Net-(D33-Pad2): track 66.0 -> 89.7 mm
- net Net-(D37-Pad2): track 88.8 -> 112.5 mm
- net Net-(D42-Pad2): track 118.7 -> 142.0 mm
- net Net-(D40-Pad2): track 106.1 -> 129.0 mm
- net Net-(D41-Pad2): track 112.3 -> 134.2 mm
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